File: espraw/espraw.kicad_pcb (KiCad board)
At the start: 2 copper layers, 4 parts, among them J1 Conn_01x08_Male, J2 Conn_01x06_Male, J3 Conn_01x08_Male, U1 ESP-12E

Commit message: add module
Parts:
- U1: footprint ESP8266:ESP-12E -> espfootprint:ESP-12E
- moved U1 0.06 mm to (143.5, 94.6)
Other:
- board text added: "makintechnologies"
