File: espraw/espraw.sch (KiCad schematic (older format))
At the start: 4 parts, among them J1 Conn_01x08_Male, J2 Conn_01x06_Male, J3 Conn_01x08_Male, U1 ESP-12E

Commit message: add module
Parts:
- removed U1: ESP-12E, ESP8266:ESP-12E, symbol ESP8266:ESP-12E
- added U1: ESP-12E, espfootprint:ESP-12E, symbol esp:ESP-12E
Connections:
- net at J1.1 (Pin_1): now also U1.1 (REST)
- net at J3.7 (Pin_7): now also U1.10 (GPIO15)
- net at J3.6 (Pin_6): now also U1.11 (GPIO2)
- net at J3.5 (Pin_5): now also U1.12 (GPIO0)
- net at J3.4 (Pin_4): now also U1.13 (GPIO4)
- net at J3.3 (Pin_3): now also U1.14 (GPIO5)
- net at J3.2 (Pin_2): now also U1.15 (RXD)
- net at J3.1 (Pin_1): now also U1.16 (TXD)
- net at J2.1 (Pin_1): now also U1.17 (CS0)
- net at J2.2 (Pin_2): now also U1.18 (MISO)
- net at J2.3 (Pin_3): now also U1.19 (GPIO9)
- net at J1.2 (Pin_2): now also U1.2 (ADC)
- net at J2.4 (Pin_4): now also U1.20 (GPIO10)
- net at J2.5 (Pin_5): now also U1.21 (MOSI)
- net at J2.6 (Pin_6): now also U1.22 (SCLK)
- net at J1.3 (Pin_3): now also U1.3 (CH_PD)
- net at J1.4 (Pin_4): now also U1.4 (GPIO16)
- net at J1.5 (Pin_5): now also U1.5 (GPIO14)
- net at J1.6 (Pin_6): now also U1.6 (GPIO12)
- net at J1.7 (Pin_7): now also U1.7 (GPIO13)
- net at J1.8 (Pin_8): now also U1.8 (VCC)
- net at J3.8 (Pin_8): now also U1.9 (GND)
Changed lines of the file:
@@
 $EndDescr
-$Comp
-L ESP8266:ESP-12E U1
-U 1 1 5FD74F57
-P 5450 3300
-F 0 "U1" H 5450 4065 50  0000 C CNN
-F 1 "ESP-12E" H 5450 3974 50  0000 C CNN
-F 2 "ESP8266:ESP-12E" H 5450 3300 50  0001 C CNN
-F 3 "http://l0l.org.uk/2014/12/esp8266-modules-hardware-guide-gotta-catch-em-all/" H 5450 3300 50  0001 C CNN
-	1    5450 3300
-	1    0    0    -1
-$EndComp
 $Comp
 L Connector:Conn_01x06_Male J2
@@
 	-1   0    0    -1
 $EndComp
+$Comp
+L esp:ESP-12E U1
+U 1 1 5FD810DF
+P 5450 3300
+F 0 "U1" H 5450 4065 50  0000 C CNN
+F 1 "ESP-12E" H 5450 3974 50  0000 C CNN
+F 2 "espfootprint:ESP-12E" H 5450 3300 50  0001 C CNN
+F 3 "http://l0l.org.uk/2014/12/esp8266-modules-hardware-guide-gotta-catch-em-all/" H 5450 3300 50  0001 C CNN
+	1    5450 3300
+	1    0    0    -1
+$EndComp
 $EndSCHEMATC
